Commit message: update to control the robot in position

File: src/motoman/motoman_hc10_support/urdf/hc10_control.xacro (robot description, xacro)
@@ -6,8 +6,8 @@
             <type>transmission_interface/SimpleTransmission</type>
             <joint name="joint_1_s">
-                <hardwareInterface>hardware_interface/EffortJointInterface</hardwareInterface>
+                <hardwareInterface>hardware_interface/PositionJointInterface</hardwareInterface>
             </joint>
             <actuator name="joint_1_s_motor">
-                <hardwareInterface>hardware_interface/EffortJointInterface</hardwareInterface>
+                <hardwareInterface>hardware_interface/PositionJointInterface</hardwareInterface>
                 <mechanicalReduction>1</mechanicalReduction>
             </actuator>
@@ -16,8 +16,8 @@
             <type>transmission_interface/SimpleTransmission</type>
             <joint name="joint_2_l">
-                <hardwareInterface>hardware_interface/EffortJointInterface</hardwareInterface>
+                <hardwareInterface>hardware_interface/PositionJointInterface</hardwareInterface>
             </joint>
             <actuator name="joint_2_l_motor">
-                <hardwareInterface>hardware_interface/EffortJointInterface</hardwareInterface>
+                <hardwareInterface>hardware_interface/PositionJointInterface</hardwareInterface>
                 <mechanicalReduction>1</mechanicalReduction>
             </actuator>
@@ -26,8 +26,8 @@
             <type>transmission_interface/SimpleTransmission</type>
             <joint name="joint_3_u">
-                <hardwareInterface>hardware_interface/EffortJointInterface</hardwareInterface>
+                <hardwareInterface>hardware_interface/PositionJointInterface</hardwareInterface>
             </joint>
             <actuator name="joint_3_u_motor">
-                <hardwareInterface>hardware_interface/EffortJointInterface</hardwareInterface>
+                <hardwareInterface>hardware_interface/PositionJointInterface</hardwareInterface>
                 <mechanicalReduction>1</mechanicalReduction>
             </actuator>
@@ -36,8 +36,8 @@
             <type>transmission_interface/SimpleTransmission</type>
             <joint name="joint_4_r">
-                <hardwareInterface>hardware_interface/EffortJointInterface</hardwareInterface>
+                <hardwareInterface>hardware_interface/PositionJointInterface</hardwareInterface>
             </joint>
             <actuator name="joint_4_r_motor">
-                <hardwareInterface>hardware_interface/EffortJointInterface</hardwareInterface>
+                <hardwareInterface>hardware_interface/PositionJointInterface</hardwareInterface>
                 <mechanicalReduction>1</mechanicalReduction>
             </actuator>
@@ -46,8 +46,8 @@
             <type>transmission_interface/SimpleTransmission</type>
             <joint name="joint_5_b">
-                <hardwareInterface>hardware_interface/EffortJointInterface</hardwareInterface>
+                <hardwareInterface>hardware_interface/PositionJointInterface</hardwareInterface>
             </joint>
             <actuator name="joint_5_b_motor">
-                <hardwareInterface>hardware_interface/EffortJointInterface</hardwareInterface>
+                <hardwareInterface>hardware_interface/PositionJointInterface</hardwareInterface>
                 <mechanicalReduction>1</mechanicalReduction>
             </actuator>
@@ -56,8 +56,8 @@
             <type>transmission_interface/SimpleTransmission</type>
             <joint name="joint_6_t">
-                <hardwareInterface>hardware_interface/EffortJointInterface</hardwareInterface>
+                <hardwareInterface>hardware_interface/PositionJointInterface</hardwareInterface>
             </joint>
             <actuator name="joint_6_t_motor">
-                <hardwareInterface>hardware_interface/EffortJointInterface</hardwareInterface>
+                <hardwareInterface>hardware_interface/PositionJointInterface</hardwareInterface>
                 <mechanicalReduction>1</mechanicalReduction>
             </actuator>

File: src/yaskawa_moveit/config/gazebo_motoman_hc10.urdf (robot description, URDF)
Before this commit: robot motoman_hc10, 10 links, 9 joints
Links:
- added link point_cloud_frame
- added link sensor_link
Joints:
- added joint camera_joint: type fixed, parent tool0, child sensor_link, origin xyz=0 0 0 rpy=0 -1.570796 0, axis 0 0 0, limit effort=10000 velocity=1000
- added joint cloud_joint: type fixed, parent tool0, child point_cloud_frame, origin xyz=0 0 0 rpy=0 0 -1.570796, axis 0 0 0, limit effort=10000 velocity=1000
