Commit message: update

File: src/motoman_V2/motoman_hc10_support/urdf/hc10_sensor.xacro (robot description, xacro)
@@ -4,4 +4,25 @@
         <xacro:include filename="$(find motoman_resources)/urdf/common_materials.xacro" />
         <link name="sensor_link">
+            <!-- Visual properties: This is how the link appears in simulation -->
+            <visual>
+                <origin xyz="0.01 0 0" rpy="0 0 0" />
+                <geometry>
+                    <!-- Replace 'box' with the desired shape (box, cylinder, sphere, mesh) -->
+                    <box size="0.05 0.05 0.1" />
+                </geometry>
+                <material name="green">
+                    <color rgba="0 1 0 1" />
+                </material>
+            </visual>
+            <visual>
+                <origin xyz="0.04 0 0" rpy="0 -1.570796 0" />
+                <geometry>
+                    <!-- Replace 'box' with the desired shape (box, cylinder, sphere, mesh) -->
+                    <cylinder radius="0.025" length="0.05" />
+                </geometry>
+                <material name="red">
+                    <color rgba="1 0 0 1" />
+                </material>
+            </visual>
         </link>
         <link name="point_cloud_frame">
@@ -41,4 +62,5 @@
                     <pointCloudCutoffMax>10.0</pointCloudCutoffMax>
                 </plugin>
+                <visualize>true</visualize>
             </sensor>
         </gazebo>

Commit message: script update

File: src/motoman_V2/motoman_hc10_support/urdf/hc10_sensor.xacro (robot description, xacro)
@@ -6,11 +6,13 @@
             <!-- Visual properties: This is how the link appears in simulation -->
             <visual>
-                <origin xyz="0.01 0 0" rpy="0 0 0" />
+                <origin xyz="0 0 0" rpy="0 0 0" />
                 <geometry>
                     <!-- Replace 'box' with the desired shape (box, cylinder, sphere, mesh) -->
                     <box size="0.05 0.05 0.1" />
+                    <!-- <mesh scale="0.001 0.001 0.001"
+                        filename="package://motoman_hc10_support/meshes/Kinect.stl" /> -->
                 </geometry>
                 <material name="green">
-                    <color rgba="0 1 0 1" />
+                    <color rgba="0 0 0 1" />
                 </material>
             </visual>
@@ -30,5 +32,5 @@
         <gazebo reference="sensor_link">
             <sensor name="kinect_camera" type="depth">
-                <update_rate>10</update_rate>
+                <update_rate>20</update_rate>
                 <camera>
                     <horizontal_fov>1.047198</horizontal_fov>
